Commit message: Rebase from 'upstream'

File: clearpath_platform_description/urdf/a200/a200.urdf.xacro (robot description, xacro)
@@ -148,5 +148,5 @@
           </xacro:if>
           <xacro:unless value="$(arg is_sim)">
-            <plugin>clearpath_platform/A200Hardware</plugin>
+            <plugin>clearpath_hardware_interfaces/A200Hardware</plugin>
             <param name="wheel_diameter">0.3302</param>
             <param name="max_accel">5.0</param>

File: clearpath_platform_description/urdf/dd100/dd100.urdf.xacro (robot description, xacro)
@@ -205,5 +205,5 @@
           </xacro:if>
           <xacro:unless value="$(arg is_sim)">
-            <plugin>clearpath_platform/PumaHardware</plugin>
+            <plugin>clearpath_hardware_interfaces/PumaHardware</plugin>
           </xacro:unless>
         </hardware>

File: clearpath_platform_description/urdf/dd150/dd150.urdf.xacro (robot description, xacro)
@@ -193,5 +193,5 @@
           </xacro:if>
           <xacro:unless value="$(arg is_sim)">
-            <plugin>clearpath_platform/PumaHardware</plugin>
+            <plugin>clearpath_hardware_interfaces/PumaHardware</plugin>
           </xacro:unless>
         </hardware>

File: clearpath_platform_description/urdf/do100/do100.urdf.xacro (robot description, xacro)
@@ -174,5 +174,5 @@
         </xacro:if>
         <xacro:unless value="$(arg is_sim)">
-          <plugin>clearpath_platform/PumaHardware</plugin>
+          <plugin>clearpath_hardware_interfaces/PumaHardware</plugin>
         </xacro:unless>
       </hardware>

File: clearpath_platform_description/urdf/j100/j100.urdf.xacro (robot description, xacro)
@@ -157,5 +157,5 @@
           </xacro:if>
           <xacro:unless value="$(arg is_sim)">
-            <plugin>clearpath_platform/J100Hardware</plugin>
+            <plugin>clearpath_hardware_interfaces/J100Hardware</plugin>
           </xacro:unless>
         </hardware>

File: clearpath_platform_description/urdf/links/box.urdf.xacro (robot description, xacro)
@@ -9,4 +9,10 @@
         <material name="clearpath_dark_grey"/>
       </visual>
+      <collision>
+        <geometry>
+          <box size="${size}"/>
+        </geometry>
+        <material name="clearpath_dark_grey"/>
+      </collision>
     </link>
     <joint name="${name}_joint" type="fixed">

File: clearpath_platform_description/urdf/links/cylinder.urdf.xacro (robot description, xacro)
@@ -9,4 +9,10 @@
         <material name="clearpath_dark_grey"/>
       </visual>
+      <collision>
+        <geometry>
+          <cylinder radius="${radius}" length="${length}"/>
+        </geometry>
+        <material name="clearpath_dark_grey"/>
+      </collision>
     </link>
     <joint name="${name}_joint" type="fixed">

File: clearpath_platform_description/urdf/links/mesh.urdf.xacro (robot description, xacro)
@@ -9,4 +9,10 @@
         <material name="clearpath_dark_grey"/>
       </visual>
+      <collision>
+        <geometry>
+          <mesh filename="${visual}"/>
+        </geometry>
+        <material name="clearpath_dark_grey"/>
+      </collision>
     </link>
     <joint name="${name}_joint" type="fixed">

File: clearpath_platform_description/urdf/links/sphere.urdf.xacro (robot description, xacro)
@@ -9,4 +9,10 @@
         <material name="clearpath_dark_grey"/>
       </visual>
+      <collision>
+        <geometry>
+          <sphere radius="${radius}"/>
+        </geometry>
+        <material name="clearpath_dark_grey"/>
+      </collision>
     </link>
     <joint name="${name}_joint" type="fixed">

File: clearpath_platform_description/urdf/r100/r100.urdf.xacro (robot description, xacro)
@@ -3,5 +3,5 @@
   <xacro:arg name="namespace" default="" />
   <xacro:arg name="is_sim" default="false" />
-  <xacro:arg name="gazebo_controllers" default="$(find clearpath_control)/config/do100/control.yaml"/>
+  <xacro:arg name="gazebo_controllers" default="$(find clearpath_control)/config/r100/control.yaml"/>
   <!-- Includes -->
   <xacro:include filename="$(find clearpath_platform_description)/urdf/r100/wheels/wheel.urdf.xacro"/>
@@ -271,5 +271,5 @@
         </xacro:if>
         <xacro:unless value="$(arg is_sim)">
-          <plugin>clearpath_platform/PumaHardware</plugin>
+          <plugin>clearpath_hardware_interfaces/PumaHardware</plugin>
         </xacro:unless>
       </hardware>

File: clearpath_platform_description/urdf/w200/w200.urdf.xacro (robot description, xacro)
@@ -172,5 +172,5 @@
           </xacro:if>
           <xacro:unless value="$(arg is_sim)">
-            <plugin>clearpath_platform/W200Hardware</plugin>
+            <plugin>clearpath_hardware_interfaces/W200Hardware</plugin>
             <param name="wheel_diameter">0.6</param>
           </xacro:unless>
